File: pcb/rev.A/zxuno1010.kicad_pcb (KiCad board)
At the start: 2 copper layers, 100 x 100 mm, 151 parts, among them J1 USB_B_Micro, J10 PJ-320, J11 TE 041021-4, J12 MEM2055-00-190-01-A, J13 Pin header 1x6 Pitch=2.54mm, J14 PJ-320, J15 Conn_02x07_Odd_Even, J2 Mini-DIN-6, J3 DB9-M, J4 Conn_02x05_Odd_Even, J5 DB15_Female_HighDensity_Mount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, J6 Conn_02x05_Odd_Even, J7 DB9-M, J8 Conn_01x04, J9 Conn_02x02_Odd_Even, Q1 BSS138, Q2 BSS138, Q3 BSS138, Q4 BSS138, Q5 BC817, Q6 BC817, SW1 Jumper / Pin header 1x2 Pitch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, SW2 SW_Push, SW3 SW_Push, SW4 SW_Push, U1 ESP-12E, U2 IS61C5128AL-10TLI, U3 XC6SLX9-TQG144, U4 W25Q32BV, U5 W25Q32BV, U6 AD724, U7 1117-3.3, U8 1117-1.2, X1 50 MHz, Y1 3.58 MHz, Y2 4.43 MHz

Commit message: update pcb rev.A
Parts:
- added R59: 4.7k, Resistor_SMD:R_0603_1608Metric_Pad0.98x0.95mm_HandSolder, F.Cu at (115.0, 105.4)
- C22: moved to F.Cu
- C23: moved to B.Cu
- moved C22 100.4 mm to (177.2, 127.1), turned to 0 degrees
- moved C23 100.4 mm to (106.0, 56.5), turned to -90 degrees
- moved R45 8.25 mm to (102.7, 83.8), turned to -90 degrees
- moved R46 7.25 mm to (102.7, 78.1), turned to 90 degrees
- moved D4 6.49 mm to (104.7, 83.8), turned to -90 degrees
- moved Y1 6.27 mm to (114.7, 83.8)
- moved C3 6.00 mm to (134.4, 78.6)
- moved C5 6.00 mm to (134.4, 84.6)
- moved R42 6.00 mm to (134.4, 77.1)
- moved R44 6.00 mm to (134.4, 83.1)
- moved D5 5.58 mm to (104.7, 78.1), turned to 90 degrees
- moved Y2 5.27 mm to (114.7, 78.1)
- moved C16 1.70 mm to (170.3, 68.3)
- moved C17 1.70 mm to (159.3, 68.3)
- moved C18 1.70 mm to (170.3, 77.3)
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Connections:
- C23 pad 2: +5V -> +5V_FUSE
- J10 pad S: unconnected-(J10-PadS) -> GND
- J12 pad 7: (no net) -> /SD_MISO
- J13 pad 3: +5V -> +5V_FUSE
- U3 pad 40: (no net) -> /MIC
- U3 pad 44: (no net) -> /SD_CD
Routing:
- net +3V3: track 0.00 -> 329.8 mm, vias 0 -> 25
- net GND: track 0.00 -> 190.0 mm, vias 0 -> 121
- net +5V_FUSE: track 0.00 -> 141.2 mm, vias 0 -> 9
- net +5V: track 0.00 -> 113.7 mm, vias 0 -> 1
- net /MIC: track 0.00 -> 101.7 mm
- net /AUDIO_LEFT: track 0.00 -> 100.4 mm
- net /AUDIO_RIGHT: track 0.00 -> 98.6 mm
- net +1V2: track 0.00 -> 82.4 mm, vias 0 -> 8
- net /EAR: track 0.00 -> 75.3 mm, vias 0 -> 2
- net /JOY12_PIN5: track 0.00 -> 61.7 mm, vias 0 -> 1
- net /VSYNC: track 0.00 -> 55.7 mm, vias 0 -> 6
- net /JOY12_PIN7: track 0.00 -> 55.1 mm, vias 0 -> 3
- net /~NMI: track 0.00 -> 51.1 mm
- net /CSYNC: track 0.00 -> 49.6 mm, vias 0 -> 4
- net /TDO: track 0.00 -> 45.2 mm, vias 0 -> 2
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
Commit message: update pcb rev.A
Parts:
- moved R54 2.65 mm to (138.5, 120.0), turned to 0 degrees
- moved R51 1.86 mm to (142.0, 120.0)
- moved F2 0.40 mm to (178.9, 106.9)
- moved J9 0.40 mm to (177.7, 110.6)
- moved R58 0.40 mm to (179.1, 106.8)
- moved R48 0.14 mm to (157.6, 120.0)
Routing:
- net /JOY2_LEFT: track 7.96 -> 72.4 mm
- net /JOY2_DOWN: track 24.0 -> 88.4 mm
- net /JOY2_UP: track 28.3 -> 92.6 mm
- net /JOY2_FIRE2: track 10.9 -> 70.5 mm, vias 0 -> 3
- net /JOY2_RIGHT: track 10.4 -> 68.2 mm, vias 0 -> 2
- net /JOY2_FIRE1: track 9.33 -> 65.2 mm, vias 0 -> 3
- net /JOY_FIRE2: track 7.31 -> 63.2 mm
- net /JOY_FIRE1: track 5.81 -> 58.5 mm, vias 0 -> 1
- net /JOY_RIGHT: track 14.7 -> 67.2 mm
- net /ESP_CTS: track 0.00 -> 51.8 mm, vias 0 -> 2
- net /JOY_LEFT: track 15.1 -> 66.0 mm
- net /LED: track 0.00 -> 50.2 mm, vias 0 -> 3
- net /JOY_UP: track 10.2 -> 60.4 mm
- net /MIC: track 101.7 -> 150.8 mm, vias 0 -> 8
- net /JOY_DOWN: track 8.10 -> 57.1 mm
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
Commit message: update pcb rev.A
Parts:
- R5: value x -> 4.7k
Routing:
- net +3V3: track 329.8 -> 653.7 mm, vias 25 -> 42
- net +5V: track 113.7 -> 192.2 mm, vias 1 -> 6
- net /~RESET: track 38.5 -> 110.9 mm
- net /SD_MISO: track 14.2 -> 79.9 mm, vias 0 -> 2
- net /SD_SCK: track 11.3 -> 67.6 mm, vias 0 -> 2
- net /SD_MOSI: track 12.7 -> 62.5 mm, vias 0 -> 2
- net GND: track 190.0 -> 235.7 mm, vias 121 -> 360
- net /STDN: track 47.1 -> 80.4 mm, vias 0 -> 4
- net /STDNB: track 50.2 -> 81.0 mm, vias 0 -> 4
- net /SD_CD: track 24.2 -> 50.8 mm, vias 3 -> 2
- net /PS2_CLK: track 26.8 -> 51.6 mm, vias 1 -> 2
- net /PS2_DATA: track 23.9 -> 46.8 mm, vias 1 -> 2
- net /PS2_PIN2: track 21.0 -> 42.1 mm, vias 1 -> 2
- net /PS2_PIN6: track 17.8 -> 37.8 mm, vias 1 -> 2
- net /SD_VDD: track 11.1 -> 15.0 mm
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
Commit message: update pcb rev.A
Parts:
- added C24: 100n, Capacitor_SMD:C_0603_1608Metric_Pad1.08x0.95mm_HandSolder, B.Cu at (110.2, 108.0)
- added C25: 10u, Capacitor_SMD:C_0805_2012Metric_Pad1.18x1.45mm_HandSolder, B.Cu at (110.2, 106.2)
- added C30: 100n, Capacitor_SMD:C_0603_1608Metric_Pad1.08x0.95mm_HandSolder, B.Cu at (115.3, 106.9)
- added C31: 10u, Capacitor_SMD:C_0805_2012Metric_Pad1.18x1.45mm_HandSolder, B.Cu at (115.3, 105.1)
- added C32: 22p, Capacitor_SMD:C_0603_1608Metric_Pad1.08x0.95mm_HandSolder, F.Cu at (111.0, 102.6)
- added C33: 22p, Capacitor_SMD:C_0603_1608Metric_Pad1.08x0.95mm_HandSolder, F.Cu at (114.5, 102.6)
- added C46: 1u, Capacitor_SMD:C_0603_1608Metric_Pad1.08x0.95mm_HandSolder, B.Cu at (115.7, 111.0)
- added C47: 100n, Capacitor_SMD:C_0603_1608Metric_Pad1.08x0.95mm_HandSolder, B.Cu at (115.7, 109.4)
- added C48: 100n, Capacitor_SMD:C_0603_1608Metric_Pad1.08x0.95mm_HandSolder, B.Cu at (109.2, 103.4)
- added LOGO2: graphic, my:zxuno_13x3.2, F.Cu at (150.8, 67.1)
- added R60: 2k, Resistor_SMD:R_0603_1608Metric_Pad0.98x0.95mm_HandSolder, F.Cu at (120.5, 68.6)
- added R61: 2k, Resistor_SMD:R_0603_1608Metric_Pad0.98x0.95mm_HandSolder, F.Cu at (118.5, 68.6)
- added U9: SAM2695, Package_DFN_QFN:QFN-48-1EP_6x6mm_P0.4mm_EP4.2x4.2mm, F.Cu at (112.8, 108.2)
- added Y3: 12 MHz, Crystal:Crystal_SMD_3225-4Pin_3.2x2.5mm_HandSoldering, F.Cu at (112.8, 99.5)
- C35: value 1u -> 10u; footprint Capacitor_SMD:C_0603_1608Metric_Pad1.08x0.95mm_HandSolder -> Capacitor_SMD:C_0805_2012Metric_Pad1.18x1.45mm_HandSolder
- moved R59 20.9 mm to (134.7, 112.3)
- moved LS1 0.20 mm to (188.1, 133.1)
Connections:
- C23 pad 2: +5V_FUSE -> +5V
- J13 pad 3: +5V_FUSE -> +5V
- U3 pad 43: (no net) -> /MIDI_IN
Routing:
- net +5V: track 192.2 -> 275.3 mm
- net +5V_FUSE: track 141.7 -> 67.5 mm
- net /MIDI_R: track 0.00 -> 61.8 mm, vias 0 -> 4
- net /MIDI_L: track 0.00 -> 61.6 mm, vias 0 -> 4
- net /MIDI_IN: track 0.00 -> 59.4 mm, vias 0 -> 4
- net +3V3: track 653.7 -> 708.5 mm, vias 42 -> 52
- net /~RESET: track 110.9 -> 152.8 mm, vias 3 -> 7
- net GND: track 235.7 -> 269.6 mm, vias 360 -> 390
- net Net-(C12-Pad1): track 5.45 -> 17.3 mm
- net Net-(C33-Pad2): track 0.00 -> 8.16 mm
- net Net-(C32-Pad2): track 0.00 -> 5.82 mm
- net /~OE: track 41.4 -> 36.4 mm, vias 0 -> 2
- net Net-(C13-Pad1): track 5.25 -> 9.93 mm
- net Net-(C30-Pad2): track 0.00 -> 3.20 mm, vias 0 -> 1
- net Net-(C24-Pad2): track 0.00 -> 3.12 mm, vias 0 -> 1
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Other:
- board text added: "ZX-UNO.1010 PCB Rev.A Eugene Lozovoy 2021"
- board text removed: "PCB Rev.A Eugene Lozovoy 2021"
- board text removed: "ZXUNO.1010"

Commit message: update pcb rev.A
Parts:
- U2: value IS61C5128AL-10TLI -> IS61WV20488BLL-10
- U4, U5: value W25Q32BV -> W25Q128
Changed lines of the file:
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@@
       (effects (font (size 1.1 0.8) (thickness 0.14)))
     )
-    (fp_text value "W25Q32BV" (at 0 3.56 90 unlocked) (layer "F.Fab")
+    (fp_text value "W25Q128" (at 0 3.56 90 unlocked) (layer "F.Fab")
       (effects (font (size 1 1) (thickness 0.15)))
     )
@@
     (fp_line (start -2.615 -1.615) (end -1.615 -2.615) (layer "F.Fab") (width 0.1))
     (pad "1" smd roundrect locked (at -3.1 -1.905 270) (size 2.6 0.6) (layers "F.Cu" "F.Paste" "F.Mask") (roundrect_rratio 0.25)
-      (net 131 "/FLASH_CS0") (pinfunction "~CS") (pintype "input"))
+      (net 131 "/FLASH_CS0") (pinfunction "~CS"))
     (pad "2" smd roundrect locked (at -3.1 -0.635 270) (size 2.6 0.6) (layers "F.Cu" "F.Paste" "F.Mask") (roundrect_rratio 0.25)
-      (net 59 "/FLASH_MISO") (pinfunction "MISO") (pintype "tri_state"))
+      (net 59 "/FLASH_MISO") (pinfunction "MISO"))
     (pad "3" smd roundrect locked (at -3.1 0.635 270) (size 2.6 0.6) (layers "F.Cu" "F.Paste" "F.Mask") (roundrect_rratio 0.25)
-      (net 57 "/FLASH_WP") (pinfunction "~WP") (pintype "input"))
+      (net 57 "/FLASH_WP") (pinfunction "~WP"))
     (pad "4" smd roundrect locked (at -3.1 1.905 270) (size 2.6 0.6) (layers "F.Cu" "F.Paste" "F.Mask") (roundrect_rratio 0.25)
-      (net 1 "GND") (pinfunction "GND") (pintype "power_in"))
+      (net 1 "GND") (pinfunction "GND"))
     (pad "5" smd roundrect locked (at 3.1 1.905 270) (size 2.6 0.6) (layers "F.Cu" "F.Paste" "F.Mask") (roundrect_rratio 0.25)
-      (net 58 "/FLASH_MOSI") (pinfunction "MOSI") (pintype "input"))
+      (net 58 "/FLASH_MOSI") (pinfunction "MOSI"))
     (pad "6" smd roundrect locked (at 3.1 0.635 270) (size 2.6 0.6) (layers "F.Cu" "F.Paste" "F.Mask") (roundrect_rratio 0.25)
-      (net 60 "/FLASH_SCK") (pinfunction "SCK") (pintype "input"))
+      (net 60 "/FLASH_SCK") (pinfunction "SCK"))
     (pad "7" smd roundrect locked (at 3.1 -0.635 270) (size 2.6 0.6) (layers "F.Cu" "F.Paste" "F.Mask") (roundrect_rratio 0.25)
-      (net 56 "/FLASH_HOLD") (pinfunction "~HOLD") (pintype "input"))
+      (net 56 "/FLASH_HOLD") (pinfunction "~HOLD"))
     (pad "8" smd roundrect locked (at 3.1 -1.905 270) (size 2.6 0.6) (layers "F.Cu" "F.Paste" "F.Mask") (roundrect_rratio 0.25)
-      (net 6 "+3V3") (pinfunction "VCC") (pintype "power_in"))
+      (net 6 "+3V3") (pinfunction "VCC"))
     (model "${KISYS3DMOD}/Package_SO.3dshapes/SO-8_5.3x6.2mm_P1.27mm.wrl"
       (offset (xyz 0 0 0))
@@
       (effects (font (size 1.1 0.8) (thickness 0.14)))
     )
-    (fp_text value "IS61C5128AL-10TLI" (at 0 10.16 unlocked) (layer "F.Fab")
+    (fp_text value "IS61WV20488BLL-10" (at 0 10.16 unlocked) (layer "F.Fab")
       (effects (font (size 1 1) (thickness 0.15)))
     )
@@
       (effects (font (size 1.1 0.8) (thickness 0.14)))
     )
-    (fp_text value "W25Q32BV" (at 0 3.56 90 unlocked) (layer "F.Fab")
+    (fp_text value "W25Q128" (at 0 3.56 90 unlocked) (layer "F.Fab")
       (effects (font (size 1 1) (thickness 0.15)))
     )
