File: pcb/rev.A/zxuno1010.kicad_pcb (KiCad board)
At the start: 2 copper layers, 100 x 100 mm, 166 parts, among them J1 USB_B_Micro, J10 PJ-320, J11 TE 041021-4, J12 MEM2055-00-190-01-A, J13 Pin header 1x6 Pitch=2.54mm, J14 PJ-320, J15 Conn_02x07_Odd_Even, J2 Mini-DIN-6, J3 DB9-M, J4 Conn_02x05_Odd_Even, J5 DB15_Female_HighDensity_Mount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, J6 Conn_02x05_Odd_Even, J7 DB9-M, J8 Conn_01x04, J9 Conn_02x02_Odd_Even, Q1 BSS138, Q2 BSS138, Q3 BSS138, Q4 BSS138, Q5 BC817, Q6 BC817, SW1 Jumper / Pin header 1x2 Pitch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, SW2 SW_Push, SW3 SW_Push, SW4 SW_Push, U1 ESP-12E, U2 IS61WV20488BLL-10, U3 XC6SLX9-TQG144, U4 W25Q128, U5 W25Q128, U6 AD724, U7 1117-3.3, U8 1117-1.2, U9 SAM2695, X1 50 MHz, Y1 3.58 MHz, Y2 4.43 MHz, Y3 12 MHz

Commit message: update pcb rev.A
Parts:
- added Q7: BC856, Package_TO_SOT_SMD:SOT-23, B.Cu at (129.5, 137.1)
- moved R14 7.40 mm to (154.2, 82.8)
- moved R16 7.40 mm to (154.2, 75.3)
- moved R17 7.40 mm to (149.1, 82.8)
- moved R19 7.40 mm to (149.1, 75.3)
- moved R20 7.40 mm to (144.0, 82.8)
- moved R22 7.40 mm to (144.0, 75.3)
- moved R29 7.40 mm to (154.2, 84.6)
- moved R31 7.40 mm to (154.2, 77.2)
- moved R32 7.40 mm to (149.1, 84.6)
- moved R37 7.40 mm to (149.1, 77.2)
- moved R38 7.40 mm to (144.0, 84.6)
- moved R41 7.40 mm to (144.0, 77.2)
- moved J2 1.25 mm to (187.4, 53.1)
- moved J15 0.65 mm to (102.5, 95.0)
- moved C12 0.50 mm to (130.4, 64.8)
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Connections:
- net /FLASH_CS renamed /~FLASH_CS
- net /FLASH_CS0 renamed /~FLASH_CS0
- net /FLASH_CS1 renamed /~FLASH_CS1
- net /FLASH_HOLD renamed /~FLASH_HOLD
- net /FLASH_WP renamed /~FLASH_WP
- net /SD_CD renamed /~SD_CD
- J11 pad 1: /SD_CS -> /~SD_CS
- J12 pad 2: /SD_CS -> /~SD_CS
- R14 pad 1: /R0 -> /R2
- R16 pad 1: /R2 -> /R0
- R17 pad 1: /G0 -> /G2
- R19 pad 1: /G2 -> /G0
- R20 pad 1: /B0 -> /B2
- R22 pad 1: /B2 -> /B0
- R29 pad 1: /R0 -> /R2
- R31 pad 1: /R2 -> /R0
- R32 pad 1: /G0 -> /G2
- R34 pad 2: /SD_CS -> Net-(R34-Pad2)
- R37 pad 1: /G2 -> /G0
- R38 pad 1: /B0 -> /B2
- R41 pad 1: /B2 -> /B0
- U3 pad 59: /SD_CS -> /~SD_CS
Routing:
- net /~SD_CS: track 0.00 -> 68.0 mm, vias 0 -> 3
- net /SD_CS: track 66.8 -> 0.00 mm, vias 3 -> 0
- net Net-(R34-Pad2): track 0.00 -> 2.90 mm
- net +3V3: track 708.5 -> 711.3 mm, vias 52 -> 51
- net GND: track 269.6 -> 267.2 mm, vias 390 -> 393
- net Net-(J2-Pad5): track 12.0 -> 13.3 mm
- net Net-(J2-Pad2): track 24.6 -> 25.8 mm
- net Net-(J2-Pad1): track 19.4 -> 20.7 mm
- net /TDO: track 45.4 -> 46.4 mm
- net /TDI: track 40.8 -> 41.9 mm
- net /TCK: track 36.7 -> 37.8 mm
- net +5V_FUSE: track 67.5 -> 68.2 mm
- net /TMS: track 39.2 -> 39.8 mm
- net /STDN: track 80.4 -> 81.0 mm
- net Net-(J2-Pad6): track 29.2 -> 29.7 mm
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
Commit message: update pcb rev.A
Parts:
- moved SW1 8.16 mm to (164.0, 60.2)
- moved C22 3.52 mm to (179.0, 130.1), turned to -90 degrees
- moved J5 2.70 mm to (145.6, 54.7)
- moved R26 2.44 mm to (174.9, 130.2), turned to -90 degrees
- moved LOGO2 2.25 mm to (150.8, 64.9)
- moved R13 1.38 mm to (158.2, 52.6)
- moved C2 1.29 mm to (176.8, 130.2), turned to 90 degrees
- moved J10 1.25 mm to (110.8, 53.4)
- moved J14 1.25 mm to (127.7, 53.4)
- moved C6 1.15 mm to (139.9, 64.8)
- moved J3 0.98 mm to (186.8, 116.1)
- moved J7 0.98 mm to (186.8, 83.9)
- moved J4 0.68 mm to (196.0, 115.7)
- moved J6 0.68 mm to (193.4, 73.3)
- moved Q5 0.30 mm to (175.9, 134.1)
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Routing:
- net Net-(J1-Pad1): track 6.20 -> 15.8 mm
- net +5V: track 274.9 -> 268.7 mm
- net /JOY12_PIN7: track 56.5 -> 62.2 mm, vias 2 -> 3
- net GND: track 267.2 -> 273.0 mm, vias 393 -> 394
- net Net-(Q5-Pad1): track 5.93 -> 2.01 mm
- net +5V_FUSE: track 68.2 -> 64.5 mm, vias 9 -> 7
- net /JOY12_PIN5: track 63.9 -> 67.6 mm
- net /HS: track 21.0 -> 23.9 mm
- net /B: track 29.8 -> 32.5 mm
- net /VS: track 20.4 -> 23.0 mm
- net /R: track 33.1 -> 35.5 mm
- net /G: track 32.0 -> 34.3 mm
- net /JOY_DOWN: track 57.1 -> 59.0 mm
- net /TAPE_IN: track 20.5 -> 22.4 mm
- net +3V3: track 711.3 -> 713.1 mm
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
Commit message: update pcb rev.A
Parts:
- added C49: 47u, Capacitor_SMD:CP_Elec_5x5.9, F.Cu at (154.8, 64.8)
- added J1: Mini-DIN-6, my:MINI_DIN_6_33PRIMARY, F.Cu at (111.0, 53.1)
- J10: value PJ-320 -> Conn_01x03; footprint my:PJ-320A_D -> Connector_PinHeader_2.54mm:PinHeader_1x03_P2.54mm_Vertical
- moved LOGO1 23.4 mm to (149.1, 88.2)
- moved JP1 13.7 mm to (102.5, 116.3), turned to 90 degrees
- moved C29 12.0 mm to (111.2, 67.3), turned to 180 degrees
- moved C14 9.56 mm to (101.4, 61.4), turned to -90 degrees
- moved R52 8.90 mm to (101.4, 68.6)
- moved D6 8.77 mm to (120.8, 63.2), turned to 90 degrees
- moved J10 8.25 mm to (108.5, 61.4), turned to 90 degrees
- moved R49 6.36 mm to (101.4, 65.0), turned to 90 degrees
- moved R54 6.00 mm to (114.6, 68.6), turned to -90 degrees
- moved C16 5.61 mm to (111.0, 68.6), turned to -90 degrees
- moved R51 4.74 mm to (103.2, 68.6), turned to -90 degrees
- moved R57 4.61 mm to (116.4, 68.6), turned to -90 degrees
- moved C15 4.61 mm to (112.8, 68.6), turned to -90 degrees
- moved R55 2.93 mm to (109.2, 68.6), turned to 90 degrees
- moved J13 2.41 mm to (104.7, 65.0), turned to 90 degrees
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- renumbered C32 to C10, C33 to C11, C6 to C12, C7 to C13, C8 to C14, C9 to C15, C10 to C16, C11 to C17, C12 to C18, C13 to C19, C14 to C20, C15 to C21, C16 to C22, C17 to C23, C18 to C24, C19 to C25, C20 to C26, C21 to C27, C22 to C28, C23 to C29, C24 to C3, C26 to C30, C27 to C31, C28 to C32, C29 to C33, C25 to C4, C3 to C5, C4 to C6, C5 to C7, C30 to C8, C31 to C9, J1 to J16, J8 to J3, J3 to J4, J4 to J5, J5 to J7, J7 to J8, LOGO2 to LOGO1, LOGO1 to LOGO2, Q2 to Q1, Q1 to Q2, Q4 to Q3, Q3 to Q4, Q7 to Q5, Q5 to Q6, Q6 to Q7, R12 to R1, R6 to R10, R9 to R11, R8 to R12, R59 to R13, R34 to R14, R35 to R15, R36 to R16, R23 to R17, R26 to R18, R13 to R19, R10 to R2, R14 to R20, R15 to R21, R16 to R22, R17 to R23, R18 to R24, R19 to R25, R20 to R26, R21 to R27, R22 to R28, R58 to R29, R11 to R3, R24 to R30, R25 to R31, R27 to R32, R28 to R33, R29 to R34, R30 to R35, R31 to R36, R32 to R37, R33 to R38, R37 to R39, R2 to R4, R38 to R40, R39 to R41, R40 to R42, R41 to R43, R42 to R44, R43 to R45, R44 to R46, R45 to R47, R46 to R48, R47 to R49, R1 to R5, R48 to R50, R49 to R51, R50 to R52, R51 to R53, R52 to R54, R53 to R55, R54 to R56, R55 to R57, R60 to R58, R61 to R59, R4 to R6, R56 to R60, R57 to R61, R3 to R7, R5 to R8, R7 to R9, SW2 to SW1, SW3 to SW2, SW4 to SW3, SW1 to SW4, U9 to U6, U6 to U7, U7 to U8, U8 to U9, Y3 to Y1, Y1 to Y2, Y2 to Y3
Connections:
- net /PS2_CLK renamed /PS2K_CLK
- net /PS2_DATA renamed /PS2K_DATA
- net /PS2_PIN2 renamed /PS2M_DATA
- net /PS2_PIN6 renamed /PS2M_CLK
- J2 pad 2: Net-(J2-Pad2) -> (no net)
- J2 pad 6: Net-(J2-Pad6) -> (no net)
- JP1 pad 1: Net-(JP1-Pad1) -> GND
- JP1 pad 2: GND -> Net-(JP1-Pad2)
- Q1 pad 3: Net-(J2-Pad5) -> Net-(J1-Pad5)
- Q2 pad 3: Net-(J2-Pad1) -> Net-(J1-Pad1)
- Q3 pad 3: Net-(J2-Pad6) -> Net-(J2-Pad5)
- Q4 pad 3: Net-(J2-Pad2) -> Net-(J2-Pad1)
- R11 pad 1: Net-(J2-Pad6) -> Net-(J2-Pad5)
- R12 pad 1: Net-(J2-Pad2) -> Net-(J2-Pad1)
- R6 pad 1: Net-(J2-Pad5) -> Net-(J1-Pad5)
- R7 pad 1: Net-(J2-Pad1) -> Net-(J1-Pad1)
- U1 pad 18: Net-(JP1-Pad1) -> Net-(JP1-Pad2)
Routing:
- net Net-(J1-Pad1): track 0.00 -> 96.6 mm, vias 0 -> 2
- net Net-(J1-Pad5): track 0.00 -> 95.0 mm, vias 0 -> 2
- net +5V_FUSE: track 64.5 -> 116.2 mm
- net Net-(J2-Pad6): track 29.7 -> 0.00 mm
- net Net-(J2-Pad2): track 25.8 -> 0.00 mm
- net Net-(J2-Pad5): track 13.3 -> 28.3 mm, vias 0 -> 1
- net Net-(JP1-Pad2): track 0.00 -> 14.6 mm, vias 0 -> 2
- net /TAPE_IN: track 22.4 -> 9.88 mm
- net Net-(C15-Pad1): track 6.99 -> 16.6 mm
- net +3V3: track 713.1 -> 706.7 mm
- net +5V: track 268.7 -> 274.1 mm, vias 6 -> 7
- net /MIC: track 149.2 -> 143.8 mm
- net Net-(J2-Pad1): track 20.7 -> 24.8 mm
- net Net-(JP1-Pad1): track 3.17 -> 0.00 mm
- net /TAPE_OUT: track 9.92 -> 12.9 mm, vias 1 -> 0
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
Commit message: update pcb rev.A
Parts:
- added R17: 220, Resistor_SMD:R_0603_1608Metric_Pad0.98x0.95mm_HandSolder, F.Cu at (116.5, 117.1)
- added R18: 220, Resistor_SMD:R_0603_1608Metric_Pad0.98x0.95mm_HandSolder, B.Cu at (137.5, 119.9)
- added R19: 220, Resistor_SMD:R_0603_1608Metric_Pad0.98x0.95mm_HandSolder, B.Cu at (193.9, 140.0)
- added R22: 220, Resistor_SMD:R_0603_1608Metric_Pad0.98x0.95mm_HandSolder, B.Cu at (184.0, 84.2)
- added R25: 220, Resistor_SMD:R_0603_1608Metric_Pad0.98x0.95mm_HandSolder, B.Cu at (184.0, 80.8)
- added R28: 220, Resistor_SMD:R_0603_1608Metric_Pad0.98x0.95mm_HandSolder, B.Cu at (184.0, 77.4)
- added R35: 220, Resistor_SMD:R_0603_1608Metric_Pad0.98x0.95mm_HandSolder, B.Cu at (184.0, 75.6)
- added R37: 10k, Resistor_SMD:R_0603_1608Metric_Pad0.98x0.95mm_HandSolder, F.Cu at (179.1, 105.6)
- added R38: 220, Resistor_SMD:R_0603_1608Metric_Pad0.98x0.95mm_HandSolder, B.Cu at (158.9, 119.8)
- added R39: 220, Resistor_SMD:R_0603_1608Metric_Pad0.98x0.95mm_HandSolder, B.Cu at (184.0, 82.5)
- added R40: 220, Resistor_SMD:R_0603_1608Metric_Pad0.98x0.95mm_HandSolder, B.Cu at (184.0, 79.1)
- added R43: 220, Resistor_SMD:R_0603_1608Metric_Pad0.98x0.95mm_HandSolder, B.Cu at (183.4, 140.0)
- moved C13 1.28 mm to (119.1, 81.8)
- moved J9 0.36 mm to (177.7, 111.0)
- moved R32 0.36 mm to (179.1, 107.2)
- moved F2 0.36 mm to (178.9, 107.2)
- moved LOGO1 0.05 mm to (149.1, 88.2)
- renumbered C49 to C26, C26 to C27, C27 to C28, C28 to C29, C29 to C30, C30 to C31, C31 to C32, C32 to C33, C33 to C34, C34 to C35, C35 to C36, C36 to C37, C37 to C38, C38 to C39, C39 to C40, C40 to C41, C41 to C42, C42 to C43, C43 to C44, C44 to C45, C45 to C46, C46 to C47, C47 to C48, C48 to C49, R17 to R20, R18 to R21, R19 to R23, R20 to R24, R21 to R26, R22 to R27, R23 to R29, R24 to R30, R25 to R31, R29 to R32, R26 to R33, R27 to R34, R28 to R36, R30 to R41, R31 to R42, R32 to R44, R33 to R45, R34 to R46, R35 to R47, R36 to R48, R37 to R49, R38 to R50, R39 to R51, R40 to R52, R41 to R53, R42 to R54, R43 to R55, R44 to R56, R45 to R57, R46 to R58, R47 to R59, R48 to R60, R49 to R61, R50 to R62, R51 to R63, R52 to R64, R53 to R65, R54 to R66, R55 to R67, R56 to R68, R57 to R69, R58 to R70, R59 to R71, R60 to R72, R61 to R73
Connections:
- J9 pad 1: Net-(J9-Pad1) -> /JOY12_SEL
- R32 pad 1: /JOY12_SEL -> Net-(R32-Pad1)
- R32 pad 2: Net-(J9-Pad1) -> /JOY12_SEL
- U3 pad 12: /ESP_TX -> Net-(R17-Pad2)
- U3 pad 14: /SD_WP -> Net-(R18-Pad2)
- U3 pad 15: /~NMI -> Net-(R19-Pad2)
- U3 pad 26: /JOY2_UP -> Net-(R22-Pad1)
- U3 pad 30: /JOY2_DOWN -> Net-(R25-Pad1)
- U3 pad 34: /JOY2_LEFT -> Net-(R28-Pad1)
- U3 pad 35: (no net) -> /MIC
- U3 pad 39: /JOY12_SEL -> Net-(R32-Pad1)
- U3 pad 40: /MIC -> (no net)
- U3 pad 41: /JOY2_RIGHT -> Net-(R35-Pad1)
- U3 pad 44: /~SD_CD -> Net-(R38-Pad1)
- U3 pad 46: /JOY2_FIRE1 -> Net-(R39-Pad1)
- U3 pad 47: /JOY2_FIRE2 -> Net-(R40-Pad1)
- U3 pad 56: /~SERVICE -> Net-(R43-Pad2)
Routing:
- net /~NMI: track 73.7 -> 4.69 mm, vias 4 -> 0
- net Net-(R28-Pad1): track 0.00 -> 67.4 mm, vias 0 -> 1
- net Net-(R22-Pad1): track 0.00 -> 65.0 mm, vias 0 -> 1
- net Net-(R25-Pad1): track 0.00 -> 64.7 mm, vias 0 -> 1
- net Net-(R19-Pad2): track 0.00 -> 64.3 mm, vias 0 -> 5
- net /JOY2_DOWN: track 88.8 -> 25.8 mm
- net /JOY2_UP: track 93.3 -> 30.4 mm
- net /JOY2_LEFT: track 72.8 -> 9.94 mm
- net Net-(R35-Pad1): track 0.00 -> 57.8 mm, vias 0 -> 3
- net /~SERVICE: track 61.0 -> 4.95 mm, vias 2 -> 0
- net /JOY2_RIGHT: track 67.3 -> 12.0 mm, vias 2 -> 0
- net Net-(R43-Pad2): track 0.00 -> 52.8 mm, vias 0 -> 3
- net Net-(R40-Pad1): track 0.00 -> 52.3 mm, vias 0 -> 3
- net /JOY2_FIRE1: track 65.7 -> 13.8 mm, vias 3 -> 0
- net /JOY2_FIRE2: track 69.9 -> 18.3 mm, vias 3 -> 0
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