File: pcb/rev.A/zxuno1010.kicad_pcb (KiCad board)
At the start: 2 copper layers, 100 x 100 mm, 181 parts, among them J1 Mini-DIN-6, J10 Conn_01x03, J11 TE 041021-4, J12 MEM2055-00-190-01-A, J13 Pin header 1x6 Pitch=2.54mm, J14 PJ-320, J15 Conn_02x07_Odd_Even, J16 USB_B_Micro, J2 Mini-DIN-6, J3 Conn_01x04, J4 DB9-M, J5 Conn_02x05_Odd_Even, J6 Conn_02x05_Odd_Even, J7 DB15_Female_HighDensity_Mount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, J8 DB9-M, J9 Conn_02x02_Odd_Even, Q1 BSS138, Q2 BSS138, Q3 BSS138, Q4 BSS138, Q5 BC856, Q6 BC817, Q7 BC817, SW1 SW_Push, SW2 SW_Push, SW3 SW_Push, SW4 Jumper / Pin header 1x2 Pitch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, U1 ESP-12E, U2 IS61WV20488BLL-10, U3 XC6SLX9-TQG144, U4 W25Q128, U5 W25Q128, U6 SAM2695, U7 AD724, U8 1117-3.3, U9 1117-1.2, X1 50 MHz, Y1 12 MHz, Y2 3.58 MHz, Y3 4.43 MHz

Commit message: update pcb rev.A
Parts:
- H1, H2, H3, H4: footprint MountingHole:MountingHole_3.2mm_M3_ISO14580 -> my:MountingHole_3.2mm_M3_dk5.2mm
- J10: value Conn_01x03 -> PJ392
- SW4: value Jumper / Pin header 1x2 Pitch=2.54mm -> PB05A
- moved SW1 0.42 mm to (172.2, 144.6)
- moved SW2 0.42 mm to (196.2, 144.6)
- moved C1 0.41 mm to (169.9, 139.0)
- moved R1 0.41 mm to (169.9, 142.0)
- moved R19 0.41 mm to (193.9, 140.4)
- moved R2 0.41 mm to (193.9, 142.0)
- moved R3 0.41 mm to (183.4, 142.0)
- moved R43 0.41 mm to (183.4, 140.4)
- moved SW3 0.41 mm to (185.7, 144.6)
Routing:
- net +3V3: track 708.8 -> 706.0 mm
- net /ESP_RX: track 45.7 -> 44.8 mm
- net Net-(JP1-Pad2): track 14.9 -> 14.1 mm

Commit message: update pcb rev.A
Parts:
- D2: value LED_Yellow -> LED_Blue
- H1, H2, H3, H4: footprint my:MountingHole_3.2mm_M3_dk5.2mm -> my:MountingHole_3.2mm_M3_dk5.2mm_Mask
- LOGO1: footprint my:zxuno_13x3.2 -> mygraphic:zxuno_13x3.2
- LOGO2: footprint my:black-mage2 -> mygraphic:black-mage-12.5x8.6
- X1: footprint Oscillator:Oscillator_SMD_EuroQuartz_XO91-4Pin_7.0x5.0mm_HandSoldering -> Oscillator:Oscillator_SMD_SeikoEpson_SG8002CA-4Pin_7.0x5.0mm
- moved Q5 13.1 mm to (116.4, 137.2)
- moved R3 1.50 mm to (181.9, 142.0)
- moved R43 1.50 mm to (181.9, 140.4)
- moved SW3 1.50 mm to (184.2, 144.6)
- moved J14 0.15 mm to (127.7, 53.3)
Connections:
- Q5 pad 1: /~SD_CS -> /ESP_TX
- R14 pad 2: Net-(Q5-Pad2) -> /LED
- R15 pad 2: /LED -> Net-(Q5-Pad2)
Routing:
- net /ESP_TX: track 11.7 -> 39.2 mm, vias 0 -> 1
- net /~SD_CS: track 68.2 -> 43.4 mm, vias 3 -> 2
- net /LED: track 50.2 -> 38.7 mm
- net +3V3: track 706.0 -> 703.7 mm
- net Net-(R19-Pad2): track 64.5 -> 63.6 mm
- net Net-(R43-Pad2): track 53.0 -> 52.4 mm
- net /MIC: track 137.3 -> 136.7 mm
Other:
- board text added: "1010"

Commit message: update pcb rev.A
Parts:
- J10: value PJ392 -> PJ-392
- J13: value Pin header 1x6 Pitch=2.54mm -> MH-M18
- J9: value Conn_02x02_Odd_Even -> Jumper
- JP1: value Jumper_NO_Small -> Jumper
- JP2: value Jumper_3_Bridged12 -> Jumper
- Y1: footprint Crystal:Crystal_SMD_3225-4Pin_3.2x2.5mm_HandSoldering -> Crystal:Crystal_SMD_SeikoEpson_TSX3225-4Pin_3.2x2.5mm_HandSoldering
Other:
- board text added: "Install one of: J11 OR J12"
- board text added: "Install one of: J4 OR J5"
- board text added: "Install one of: J8 OR J6"
