File: pcb/rev.A/zxuno1010.kicad_sch (KiCad schematic)
At the start: 152 parts, among them J1 USB_B_Micro, J10 PJ-320, J11 TE 041021-4, J12 MEM2055-00-190-01-A, J13 Pin header 1x6 Pitch=2.54mm, J14 PJ-320, J15 Conn_02x07_Odd_Even, J2 Mini-DIN-6, J3 DB9-M, J4 Conn_02x05_Odd_Even, J5 DB15_Female_HighDensity_Mount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, J6 Conn_02x05_Odd_Even, J7 DB9-M, J8 Conn_01x04, J9 Conn_02x02_Odd_Even, Q1 BSS138, Q2 BSS138, Q3 BSS138, Q4 BSS138, Q5 BC817, Q6 BC817, SW1 Jumper / Pin header 1x2 Pitch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, SW2 SW_Push, SW3 SW_Push, SW4 SW_Push, U1 ESP-12E, U2 IS61C5128AL-10TLI, U3 XC6SLX9-TQG144, U4 W25Q32BV, U5 W25Q32BV, U6 AD724, U7 1117-3.3, U8 1117-1.2, X1 50 MHz, Y1 3.58 MHz, Y2 4.43 MHz

Commit message: update pcb rev.A
Parts:
- added R59: 4.7k, Resistor_SMD:R_0603_1608Metric_Pad0.98x0.95mm_HandSolder, symbol Device:R
Connections:
- net MISO is gone; now on net SD_MISO: J12.7 (DAT0)
- net +5V: no longer C23.2, J13.3 (Pin_3)
- net +5V_FUSE: now also C23.2, J13.3 (Pin_3)
- net GND: now also J10.S, R59.2
- net MIC: now also U3.40 (IO_L64N_D9_2)
- net SD_CD: now also U3.44 (IO_L62P_D5_2)
- net ~OE: now also R59.1
- no-connect marks 47 -> 44
Other:
- moved on the sheet: D1, D2, D3, R34, R35, R36

Commit message: update pcb rev.A
Parts:
- R5: value x -> 4.7k
Other:
- moved on the sheet: J4, J6, J9, R58

Commit message: update pcb rev.A
Parts:
- added C24, C30, C47, C48: 100n, Capacitor_SMD:C_0603_1608Metric_Pad1.08x0.95mm_HandSolder, symbol Device:C
- added C25, C31: 10u, Capacitor_SMD:C_0805_2012Metric_Pad1.18x1.45mm_HandSolder, symbol Device:C
- added C32, C33: 22p, Capacitor_SMD:C_0603_1608Metric_Pad1.08x0.95mm_HandSolder, symbol Device:C
- added C46: 1u, Capacitor_SMD:C_0603_1608Metric_Pad1.08x0.95mm_HandSolder, symbol Device:C
- added LOGO2: graphic, my:zxuno_13x3.2, symbol my:logo
- added R60, R61: 2k, Resistor_SMD:R_0603_1608Metric_Pad0.98x0.95mm_HandSolder, symbol Device:R
- added U9: SAM2695, Package_DFN_QFN:QFN-48-1EP_6x6mm_P0.4mm_EP4.2x4.2mm, symbol my:SAM2695
- added Y3: 12 MHz, Crystal:Crystal_SMD_3225-4Pin_3.2x2.5mm_HandSoldering, symbol Device:Crystal_GND24
- C35: value 1u -> 10u; footprint Capacitor_SMD:C_0603_1608Metric_Pad1.08x0.95mm_HandSolder -> Capacitor_SMD:C_0805_2012Metric_Pad1.18x1.45mm_HandSolder
- LOGO1: now left out of the parts list
Connections:
- net +3V3: now also C46.2, C47.2, C48.2, U9.11 (VD33), U9.12 (~WR), U9.20 (VD33), U9.31 (VD33), U9.35 (VD33), U9.41 (VD33), U9.46 (VD33), U9.47 (XDIV), U9.6 (VA33), U9.8 (VD33)
- net +5V: now also C23.2, J13.3 (Pin_3)
- net +5V_FUSE: no longer C23.2, J13.3 (Pin_3)
- net GND: now also C24.1, C25.1, C30.1, C31.1, C32.1, C33.1, C46.1, C47.1, C48.1, U9.10 (A0), U9.13 (GND), U9.14 (~CS), U9.15 (~RD), U9.18 (GND), U9.25 (GND), U9.36 (GND), U9.4 (AGND), U9.45 (GND), U9.48 (GND), U9.49 (GND), U9.7 (MICIN), U9.9 (GND), Y3.2, Y3.4
- net ~RESET: now also U9.38 (~RST~/~PD~)
- net at C12.1, C14.1, R56.2: now also R60.2
- net MIDI_IN: now reaches U3.43 (IO_L62N_D6_2)
- net MIDI_IN: now also U9.16 (MIDI_IN)
- net at C13.1, C15.1, R57.2: now also R61.2
- new net: C32.2, U9.40 (X2), Y3.1
- new net: C33.2, U9.39 (X1), Y3.3
- new net: C24.2, C25.2, U9.5 (VCM)
- new net: C30.2, C31.2, U9.34 (OUTVC12)
- new net MIDI_L: R60.1, U9.1 (AOUTL)
- new net MIDI_R: R61.1, U9.2 (AOUTR)
- no-connect marks 44 -> 54
Other:
- note added: "MIDI"
- moved on the sheet: C1, C12, C13, C14, C15, C2, C23, C26, C27, C28, C29, C34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

Commit message: update pcb rev.A
Parts:
- U2: value IS61C5128AL-10TLI -> IS61WV20488BLL-10
- U4, U5: value W25Q32BV -> W25Q128
Other:
- moved on the sheet: C31, C32, C33, D4, D5

Commit message: update pcb rev.A
Parts:
- added Q7: BC856, Package_TO_SOT_SMD:SOT-23, symbol Transistor_BJT:BC856
Connections:
- net B0: now also R22.1, R41.1; no longer R20.1, R38.1
- net B2: now also R20.1, R38.1; no longer R22.1, R41.1
- net G0: now also R19.1, R37.1; no longer R17.1, R32.1
- net G2: now also R17.1, R32.1; no longer R19.1, R37.1
- net GND: now also Q7.3 (C)
- net R0: now also R16.1, R31.1; no longer R14.1, R29.1
- net R2: now also R14.1, R29.1; no longer R16.1, R31.1
- net FLASH_CS renamed ~FLASH_CS
- net FLASH_CS0 renamed ~FLASH_CS0
- net FLASH_CS1 renamed ~FLASH_CS1
- net FLASH_HOLD renamed ~FLASH_HOLD
- net FLASH_WP renamed ~FLASH_WP
- net SD_CD renamed ~SD_CD
- net SD_CS renamed ~SD_CS
- net ~SD_CS: now also Q7.1 (B); no longer R34.2
- new net: Q7.2 (E), R34.2
Other:
- moved on the sheet: D1, D2, D3, R34, R35, R36

Commit message: update pcb rev.A
Parts:
- removed J10: PJ-320, my:PJ-320A_D, symbol Connector:AudioJack4
- added C49: 47u, Capacitor_SMD:CP_Elec_5x5.9, symbol Device:CP
- added J1: Mini-DIN-6, my:MINI_DIN_6_33PRIMARY, symbol Connector:Mini-DIN-6
- added J10: Conn_01x03, Connector_PinHeader_2.54mm:PinHeader_1x03_P2.54mm_Vertical, symbol Connector_Generic:Conn_01x03
- renumbered C32 to C10, C33 to C11, C6 to C12, C7 to C13, C8 to C14, C9 to C15, C10 to C16, C11 to C17, C12 to C18, C13 to C19, C14 to C20, C15 to C21, C16 to C22, C17 to C23, C18 to C24, C19 to C25, C20 to C26, C21 to C27, C22 to C28, C23 to C29, C24 to C3, C26 to C30, C27 to C31, C28 to C32, C29 to C33, C25 to C4, C3 to C5, C4 to C6, C5 to C7, C30 to C8, C31 to C9, J1 to J16, J8 to J3, J3 to J4, J4 to J5, J5 to J7, J7 to J8, LOGO2 to LOGO1, LOGO1 to LOGO2, Q2 to Q1, Q1 to Q2, Q4 to Q3, Q3 to Q4, Q7 to Q5, Q5 to Q6, Q6 to Q7, R12 to R1, R6 to R10, R9 to R11, R8 to R12, R59 to R13, R34 to R14, R35 to R15, R36 to R16, R23 to R17, R26 to R18, R13 to R19, R10 to R2, R14 to R20, R15 to R21, R16 to R22, R17 to R23, R18 to R24, R19 to R25, R20 to R26, R21 to R27, R22 to R28, R58 to R29, R11 to R3, R24 to R30, R25 to R31, R27 to R32, R28 to R33, R29 to R34, R30 to R35, R31 to R36, R32 to R37, R33 to R38, R37 to R39, R2 to R4, R38 to R40, R39 to R41, R40 to R42, R41 to R43, R42 to R44, R43 to R45, R44 to R46, R45 to R47, R46 to R48, R47 to R49, R1 to R5, R48 to R50, R49 to R51, R50 to R52, R51 to R53, R52 to R54, R53 to R55, R54 to R56, R55 to R57, R60 to R58, R61 to R59, R4 to R6, R56 to R60, R57 to R61, R3 to R7, R5 to R8, R7 to R9, SW2 to SW1, SW3 to SW2, SW4 to SW3, SW1 to SW4, U9 to U6, U6 to U7, U7 to U8, U8 to U9, Y3 to Y1, Y1 to Y2, Y2 to Y3
Connections:
- net +5V: now also C49.1
- net +5V_FUSE: now also J1.4
- net GND: now also JP1.1, C49.2, J1.3, J10.1 (Pin_1); no longer JP1.2
- net TAPE_IN: now also J10.2 (Pin_2)
- net TAPE_OUT: now also J10.3 (Pin_3)
- net at Q2.3 (D), R7.1: now also J1.1; no longer J2.1
- net at Q4.3 (D), R12.1: now also J2.1; no longer J2.2
- net at Q1.3 (D), R6.1: now also J1.5; no longer J2.5
- net at U1.18 (GPIO0): now also JP1.2; no longer JP1.1
- net at Q3.3 (D), R11.1: now also J2.5; no longer J2.6
- net PS2_CLK renamed PS2K_CLK
- net PS2_DATA renamed PS2K_DATA
- net PS2_PIN2 renamed PS2M_DATA
- net PS2_PIN6 renamed PS2M_CLK
- no-connect marks 54 -> 58
Other:
- moved on the sheet: J2, Q1, Q2, Q3, Q4, R10, R11, R12, R4, R5, R6, R7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

Commit message: update pcb rev.A
Parts:
- added R17, R18, R19, R22, R25, R28, R35, R38, R39, R40, R43: 220, Resistor_SMD:R_0603_1608Metric_Pad0.98x0.95mm_HandSolder, symbol Device:R
- added R37: 10k, Resistor_SMD:R_0603_1608Metric_Pad0.98x0.95mm_HandSolder, symbol Device:R
- renumbered C49 to C26, C26 to C27, C27 to C28, C28 to C29, C29 to C30, C30 to C31, C31 to C32, C32 to C33, C33 to C34, C34 to C35, C35 to C36, C36 to C37, C37 to C38, C38 to C39, C39 to C40, C40 to C41, C41 to C42, C42 to C43, C43 to C44, C44 to C45, C45 to C46, C46 to C47, C47 to C48, C48 to C49, R17 to R20, R18 to R21, R19 to R23, R20 to R24, R21 to R26, R22 to R27, R23 to R29, R24 to R30, R25 to R31, R29 to R32, R26 to R33, R27 to R34, R28 to R36, R30 to R41, R31 to R42, R32 to R44, R33 to R45, R34 to R46, R35 to R47, R36 to R48, R37 to R49, R38 to R50, R39 to R51, R40 to R52, R41 to R53, R42 to R54, R43 to R55, R44 to R56, R45 to R57, R46 to R58, R47 to R59, R48 to R60, R49 to R61, R50 to R62, R51 to R63, R52 to R64, R53 to R65, R54 to R66, R55 to R67, R56 to R68, R57 to R69, R58 to R70, R59 to R71, R60 to R72, R61 to R73
Connections:
- net +3V3: now also R37.1
- net ESP_TX: now also R17.1; no longer U3.12 (IO_L49P_3)
- net JOY12_SEL: now also J9.1 (Pin_1), R32.2, R37.2; no longer R32.1, U3.39 (IO_L65P_INIT_B_2)
- net JOY2_DOWN: now also R25.2; no longer U3.30 (IO_L36P_3)
- net JOY2_FIRE1: now also R39.2; no longer U3.46 (IO_L49P_D3_2)
- net JOY2_FIRE2: now also R40.2; no longer U3.47 (IO_L48N_RDWR_B_VREF_2)
- net JOY2_LEFT: now also R28.2; no longer U3.34 (IO_L1N_VREF_3)
- net JOY2_RIGHT: now also R35.2; no longer U3.41 (IO_L64P_D8_2)
- net JOY2_UP: now also R22.2; no longer U3.26 (IO_L37N_3)
- net MIC: now also U3.35 (IO_L1P_3); no longer U3.40 (IO_L64N_D9_2)
- net SD_WP: now also R18.1; no longer U3.14 (IO_L44N_GCLK20_3)
- net ~NMI: now also R19.1; no longer U3.15 (IO_L44P_GCLK21_3)
- net ~SD_CD: now also R38.2; no longer U3.44 (IO_L62P_D5_2)
- net ~SERVICE: now also R43.1; no longer U3.56 (IO_L30P_GCLK1_D13_2)
- new net: R39.1, U3.46 (IO_L49P_D3_2)
- new net: R35.1, U3.41 (IO_L64P_D8_2)
- new net: R22.1, U3.26 (IO_L37N_3)
- new net: R40.1, U3.47 (IO_L48N_RDWR_B_VREF_2)
- new net: R18.2, U3.14 (IO_L44N_GCLK20_3)
- new net: R38.1, U3.44 (IO_L62P_D5_2)
- new net: R28.1, U3.34 (IO_L1N_VREF_3)
- new net: R43.2, U3.56 (IO_L30P_GCLK1_D13_2)
- new net: R32.1, U3.39 (IO_L65P_INIT_B_2)
- new net: R17.2, U3.12 (IO_L49P_3)
- new net: R19.2, U3.15 (IO_L44P_GCLK21_3)
- new net: R25.1, U3.30 (IO_L36P_3)
Other:
- note added: "220 Ohm resistors are used to prevent I/O pins damage as on original ZXUNO these pins may be used for other purposes"
- moved on the sheet: JP1, R13, R32, U2

Commit message: update pcb rev.A
Parts:
- H1, H2, H3, H4: footprint MountingHole:MountingHole_3.2mm_M3_ISO14580 -> my:MountingHole_3.2mm_M3_dk5.2mm
- J10: value Conn_01x03 -> PJ392
- SW4: value Jumper / Pin header 1x2 Pitch=2.54mm -> PB05A
Other:
- note added: "JTAG"
- note added: "Screws: 4xM3 dk=5mm L=4mm"
- note removed: "Debug"
Changed lines of the file:
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@@
     (effects (font (size 1 1)) (justify left bottom))
   )
-  (text "Debug" (at 292.1 251.46 180)
+  (text "JTAG" (at 290.195 251.46 180)
     (effects (font (size 2 2) italic) (justify right bottom))
   )
@@
     (effects (font (size 2 2) italic) (justify right bottom))
   )
+  (text "Screws: 4xM3 dk=5mm L=4mm" (at 328.93 320.675 180)
+    (effects (font (size 1.27 1.27)) (justify right bottom))
+  )
   (text "For Megadrive gamepad connect 1-3 and 2-4" (at 329.565 147.955 180)
     (effects (font (size 1.27 1.27) italic) (justify right bottom))
@@
       (effects (font (size 1 1)) (justify left))
     )
-    (property "Footprint" "MountingHole:MountingHole_3.2mm_M3_ISO14580" (id 2) (at 315.595 294.64 0)
+    (property "Footprint" "my:MountingHole_3.2mm_M3_dk5.2mm" (id 2) (at 315.595 294.64 0)
       (effects (font (size 1.27 1.27)) hide)
     )
@@
       (effects (font (size 1 1)) (justify left))
     )
-    (property "Footprint" "MountingHole:MountingHole_3.2mm_M3_ISO14580" (id 2) (at 315.595 300.99 0)
+    (property "Footprint" "my:MountingHole_3.2mm_M3_dk5.2mm" (id 2) (at 315.595 300.99 0)
       (effects (font (size 1.27 1.27)) hide)
     )
@@
       (effects (font (size 1 1)) (justify left))
     )
-    (property "Footprint" "MountingHole:MountingHole_3.2mm_M3_ISO14580" (id 2) (at 315.595 307.34 0)
+    (property "Footprint" "my:MountingHole_3.2mm_M3_dk5.2mm" (id 2) (at 315.595 307.34 0)
       (effects (font (size 1.27 1.27)) hide)
     )
@@
       (effects (font (size 1 1)) (justify left))
     )
-    (property "Footprint" "MountingHole:MountingHole_3.2mm_M3_ISO14580" (id 2) (at 315.595 313.69 0)
+    (property "Footprint" "my:MountingHole_3.2mm_M3_dk5.2mm" (id 2) (at 315.595 313.69 0)
       (effects (font (size 1.27 1.27)) hide)
     )
@@
       (effects (font (size 1 1)))
     )
-    (property "Value" "Jumper / Pin header 1x2 Pitch=2.54mm" (id 1) (at 226.695 275.1074 0)
+    (property "Value" "PB05A" (id 1) (at 226.695 275.1074 0)
       (effects (font (size 1 1)) hide)
     )
@@
       (effects (font (size 1 1)) (justify left))
     )
-    (property "Value" "Conn_01x03" (id 1) (at 264.795 232.4099 0)
+    (property "Value" "PJ392" (id 1) (at 264.795 232.4099 0)
       (effects (font (size 1 1)) (justify left) hide)
     )
@@
     )
     (path "/2f8fe43d-0aef-44a9-b4e2-3b3365181bba"
-      (reference "H1") (unit 1) (value "MountingHole") (footprint "MountingHole:MountingHole_3.2mm_M3_ISO14580")
+      (reference "H1") (unit 1) (value "MountingHole") (footprint "my:MountingHole_3.2mm_M3_dk5.2mm")
     )
     (path "/35d0454f-36ff-4f88-abfb-63c692ac59f4"
-      (reference "H2") (unit 1) (value "MountingHole") (footprint "MountingHole:MountingHole_3.2mm_M3_ISO14580")
+      (reference "H2") (unit 1) (value "MountingHole") (footprint "my:MountingHole_3.2mm_M3_dk5.2mm")
     )
     (path "/94f3dbfc-30e0-4568-a542-0adfd7440004"
-      (reference "H3") (unit 1) (value "MountingHole") (footprint "MountingHole:MountingHole_3.2mm_M3_ISO14580")
+      (reference "H3") (unit 1) (value "MountingHole") (footprint "my:MountingHole_3.2mm_M3_dk5.2mm")
     )
     (path "/387d9e43-d657-41ab-8d4a-96ecdbbfa1ca"
-      (reference "H4") (unit 1) (value "MountingHole") (footprint "MountingHole:MountingHole_3.2mm_M3_ISO14580")
+      (reference "H4") (unit 1) (value "MountingHole") (footprint "my:MountingHole_3.2mm_M3_dk5.2mm")
     )
     (path "/2a36f1d7-dfe4-4a2b-86e2-bfadb83dc64c"
@@
     )
     (path "/e8c4a248-1da0-4da0-82c3-044d513b286f"
-      (reference "J10") (unit 1) (value "Conn_01x03") (footprint "Connector_PinHeader_2.54mm:PinHeader_1x03_P2.54mm_Vertical")
+      (reference "J10") (unit 1) (value "PJ392") (footprint "Connector_PinHeader_2.54mm:PinHeader_1x03_P2.54mm_Vertical")
     )
     (path "/733e0df2-b5ba-4317-b4c0-8c3f642bd2b8"
@@
     )
     (path "/1f4cf102-402d-49dc-87d6-ee27ccbec911"
-      (reference "SW4") (unit 1) (value "Jumper / Pin header 1x2 Pitch=2.54mm") (footprint "Connector_Molex:Molex_KK-254_AE-6410-02A_1x02_P2.54mm_Vertical")
+      (reference "SW4") (unit 1) (value "PB05A") (footprint "Connector_Molex:Molex_KK-254_AE-6410-02A_1x02_P2.54mm_Vertical")
     )
     (path "/c73d62ac-494b-4b06-bed5-a6d3b2e959dd"
