File: pcb/rev.A/zxuno1010.kicad_sch (KiCad schematic)
At the start: 182 parts, among them J1 Mini-DIN-6, J10 PJ392, J11 TE 041021-4, J12 MEM2055-00-190-01-A, J13 Pin header 1x6 Pitch=2.54mm, J14 PJ-320, J15 Conn_02x07_Odd_Even, J16 USB_B_Micro, J2 Mini-DIN-6, J3 Conn_01x04, J4 DB9-M, J5 Conn_02x05_Odd_Even, J6 Conn_02x05_Odd_Even, J7 DB15_Female_HighDensity_Mount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, J8 DB9-M, J9 Conn_02x02_Odd_Even, Q1 BSS138, Q2 BSS138, Q3 BSS138, Q4 BSS138, Q5 BC856, Q6 BC817, Q7 BC817, SW1 SW_Push, SW2 SW_Push, SW3 SW_Push, SW4 PB05A, U1 ESP-12E, U2 IS61WV20488BLL-10, U3 XC6SLX9-TQG144, U4 W25Q128, U5 W25Q128, U6 SAM2695, U7 AD724, U8 1117-3.3, U9 1117-1.2, X1 50 MHz, Y1 12 MHz, Y2 3.58 MHz, Y3 4.43 MHz

Commit message: update pcb rev.A
Parts:
- D2: value LED_Yellow -> LED_Blue
- H1, H2, H3, H4: footprint my:MountingHole_3.2mm_M3_dk5.2mm -> my:MountingHole_3.2mm_M3_dk5.2mm_Mask
- LOGO1: footprint my:zxuno_13x3.2 -> mygraphic:zxuno_13x3.2
- LOGO2: footprint my:black-mage2 -> mygraphic:black-mage-12.5x8.6
- X1: footprint Oscillator:Oscillator_SMD_EuroQuartz_XO91-4Pin_7.0x5.0mm_HandSoldering -> Oscillator:Oscillator_SMD_SeikoEpson_SG8002CA-4Pin_7.0x5.0mm
Connections:
- net ESP_TX: now also Q5.1 (B)
- net LED: now also R14.2; no longer R15.2
- net ~SD_CS: no longer Q5.1 (B)
- net at Q5.2 (E): now also R15.2; no longer R14.2
Other:
- moved on the sheet: D1, D2, R14, R15
Changed lines of the file:
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@@
     (effects (font (size 1 1)) (justify left bottom))
   )
-  (label "~SD_CS" (at 384.81 74.295 0)
+  (label "ESP_TX" (at 384.81 74.295 0)
     (effects (font (size 1 1)) (justify left bottom))
   )
@@
       (effects (font (size 1 1)) (justify left))
     )
-    (property "Footprint" "my:MountingHole_3.2mm_M3_dk5.2mm" (id 2) (at 315.595 294.64 0)
+    (property "Footprint" "my:MountingHole_3.2mm_M3_dk5.2mm_Mask" (id 2) (at 315.595 294.64 0)
       (effects (font (size 1.27 1.27)) hide)
     )
@@
       (effects (font (size 1 1)) (justify left))
     )
-    (property "Footprint" "my:MountingHole_3.2mm_M3_dk5.2mm" (id 2) (at 315.595 300.99 0)
+    (property "Footprint" "my:MountingHole_3.2mm_M3_dk5.2mm_Mask" (id 2) (at 315.595 300.99 0)
       (effects (font (size 1.27 1.27)) hide)
     )
@@
       (effects (font (size 1 1)) (justify left))
     )
-    (property "Footprint" "my:MountingHole_3.2mm_M3_dk5.2mm" (id 2) (at 315.595 307.34 0)
+    (property "Footprint" "my:MountingHole_3.2mm_M3_dk5.2mm_Mask" (id 2) (at 315.595 307.34 0)
       (effects (font (size 1.27 1.27)) hide)
     )
@@
       (effects (font (size 1 1)) (justify left))
     )
-    (property "Footprint" "my:MountingHole_3.2mm_M3_dk5.2mm" (id 2) (at 315.595 313.69 0)
+    (property "Footprint" "my:MountingHole_3.2mm_M3_dk5.2mm_Mask" (id 2) (at 315.595 313.69 0)
       (effects (font (size 1.27 1.27)) hide)
     )
@@
   (symbol (lib_id "Device:R") (at 408.305 77.47 0) (unit 1)
     (in_bom yes) (on_board yes)
-    (property "Reference" "R14" (id 0) (at 410.0831 76.0741 0)
+    (property "Reference" "R15" (id 0) (at 410.0831 76.0741 0)
       (effects (font (size 1 1)) (justify left))
     )
@@
   (symbol (lib_id "Device:R") (at 415.925 77.47 0) (unit 1)
     (in_bom yes) (on_board yes)
-    (property "Reference" "R15" (id 0) (at 417.7031 76.0741 0)
+    (property "Reference" "R14" (id 0) (at 417.7031 76.0741 0)
       (effects (font (size 1 1)) (justify left))
     )
@@
   (symbol (lib_id "Device:LED") (at 408.305 69.85 90) (unit 1)
     (in_bom yes) (on_board yes)
-    (property "Reference" "D1" (id 0) (at 411.48 69.85 90)
+    (property "Reference" "D2" (id 0) (at 411.48 69.85 90)
       (effects (font (size 1 1)))
     )
-    (property "Value" "LED_Red" (id 1) (at 407.035 87.63 90)
+    (property "Value" "LED_Blue" (id 1) (at 408.305 87.63 90)
       (effects (font (size 1 1)))
     )
@@
   (symbol (lib_id "Device:LED") (at 415.925 69.85 90) (unit 1)
     (in_bom yes) (on_board yes)
-    (property "Reference" "D2" (id 0) (at 419.1 69.85 90)
+    (property "Reference" "D1" (id 0) (at 419.1 69.85 90)
       (effects (font (size 1 1)))
     )
-    (property "Value" "LED_Yellow" (id 1) (at 415.925 87.63 90)
+    (property "Value" "LED_Red" (id 1) (at 415.925 87.63 90)
       (effects (font (size 1 1)))
     )
@@
       (effects (font (size 1 1)))
     )
-    (property "Value" "LED_Green" (id 1) (at 425.45 87.63 90)
+    (property "Value" "LED_Green" (id 1) (at 424.18 87.63 90)
       (effects (font (size 1 1)))
     )
@@
       (effects (font (size 1 1)) hide)
     )
-    (property "Footprint" "my:zxuno_13x3.2" (id 2) (at 270.51 309.88 0)
+    (property "Footprint" "mygraphic:zxuno_13x3.2" (id 2) (at 270.51 309.88 0)
       (effects (font (size 1.27 1.27)) hide)
     )
@@
       (effects (font (size 1 1)) hide)
     )
-    (property "Footprint" "my:black-mage2" (id 2) (at 283.21 309.88 0)
+    (property "Footprint" "mygraphic:black-mage-12.5x8.6" (id 2) (at 283.21 309.88 0)
       (effects (font (size 1.27 1.27)) hide)
     )
@@
       (effects (font (size 1 1)) (justify left))
     )
-    (property "Footprint" "Oscillator:Oscillator_SMD_EuroQuartz_XO91-4Pin_7.0x5.0mm_HandSoldering" (id 2) (at 170.18 203.835 0)
+    (property "Footprint" "Oscillator:Oscillator_SMD_SeikoEpson_SG8002CA-4Pin_7.0x5.0mm" (id 2) (at 170.18 203.835 0)
       (effects (font (size 1.27 1.27)) hide)
     )
@@
     )
     (path "/35b42faf-4604-4a4f-a642-c4bb2437cffa"
-      (reference "D2") (unit 1) (value "LED_Yellow") (footprint "LED_THT:LED_D3.0mm_Horizontal_O1.27mm_Z6.0mm")
+      (reference "D2") (unit 1) (value "LED_Blue") (footprint "LED_THT:LED_D3.0mm_Horizontal_O1.27mm_Z6.0mm")
     )
     (path "/a1d9b023-ff68-46c4-9dd0-0d3c73e90c6e"
@@
     )
     (path "/2f8fe43d-0aef-44a9-b4e2-3b3365181bba"
-      (reference "H1") (unit 1) (value "MountingHole") (footprint "my:MountingHole_3.2mm_M3_dk5.2mm")
+      (reference "H1") (unit 1) (value "MountingHole") (footprint "my:MountingHole_3.2mm_M3_dk5.2mm_Mask")
     )
     (path "/35d0454f-36ff-4f88-abfb-63c692ac59f4"
-      (reference "H2") (unit 1) (value "MountingHole") (footprint "my:MountingHole_3.2mm_M3_dk5.2mm")
+      (reference "H2") (unit 1) (value "MountingHole") (footprint "my:MountingHole_3.2mm_M3_dk5.2mm_Mask")
     )
     (path "/94f3dbfc-30e0-4568-a542-0adfd7440004"
-      (reference "H3") (unit 1) (value "MountingHole") (footprint "my:MountingHole_3.2mm_M3_dk5.2mm")
+      (reference "H3") (unit 1) (value "MountingHole") (footprint "my:MountingHole_3.2mm_M3_dk5.2mm_Mask")
     )
     (path "/387d9e43-d657-41ab-8d4a-96ecdbbfa1ca"
-      (reference "H4") (unit 1) (value "MountingHole") (footprint "my:MountingHole_3.2mm_M3_dk5.2mm")
+      (reference "H4") (unit 1) (value "MountingHole") (footprint "my:MountingHole_3.2mm_M3_dk5.2mm_Mask")
     )
     (path "/2a36f1d7-dfe4-4a2b-86e2-bfadb83dc64c"
@@
     )
     (path "/6e5402f4-28a6-421e-9862-e1d2ac04c225"
-      (reference "LOGO1") (unit 1) (value "graphic") (footprint "my:zxuno_13x3.2")
+      (reference "LOGO1") (unit 1) (value "graphic") (footprint "mygraphic:zxuno_13x3.2")
     )
     (path "/74bc78de-3bc3-4ca2-a941-3aa58a86950f"
-      (reference "LOGO2") (unit 1) (value "graphic") (footprint "my:black-mage2")
+      (reference "LOGO2") (unit 1) (value "graphic") (footprint "mygraphic:black-mage-12.5x8.6")
     )
     (path "/98f5b6b3-1608-46ad-a2ca-a387b7ba8f9e"
@@
     )
     (path "/63646a0d-c99e-4a1c-bd86-154ac3df1a0f"
-      (reference "X1") (unit 1) (value "50 MHz") (footprint "Oscillator:Oscillator_SMD_EuroQuartz_XO91-4Pin_7.0x5.0mm_HandSoldering")
+      (reference "X1") (unit 1) (value "50 MHz") (footprint "Oscillator:Oscillator_SMD_SeikoEpson_SG8002CA-4Pin_7.0x5.0mm")
     )
     (path "/1f0d16be-9630-4d59-b559-5e9a315adc32"

Commit message: update pcb rev.A
Parts:
- J10: value PJ392 -> PJ-392
- J13: value Pin header 1x6 Pitch=2.54mm -> MH-M18; Desc M18 -> (none)
- J9: value Conn_02x02_Odd_Even -> Jumper
- JP1: value Jumper_NO_Small -> Jumper
- JP2: value Jumper_3_Bridged12 -> Jumper
- Y1: footprint Crystal:Crystal_SMD_3225-4Pin_3.2x2.5mm_HandSoldering -> Crystal:Crystal_SMD_SeikoEpson_TSX3225-4Pin_3.2x2.5mm_HandSoldering
Changed lines of the file:
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@@
     (stroke (width 0) (type solid) (color 0 0 0 0))
   )
-  (wire (pts (xy 33.02 240.03) (xy 33.02 248.92))
-    (stroke (width 0) (type solid) (color 0 0 0 0))
-  )
   (wire (pts (xy 33.655 78.105) (xy 34.925 78.105))
     (stroke (width 0) (type solid) (color 0 0 0 0))
@@
     (stroke (width 0) (type solid) (color 0 0 0 0))
   )
-  (wire (pts (xy 34.925 238.76) (xy 34.925 240.03))
+  (wire (pts (xy 34.925 238.76) (xy 34.925 248.92))
     (stroke (width 0) (type solid) (color 0 0 0 0))
   )
@@
     (stroke (width 0) (type solid) (color 0 0 0 0))
   )
-  (wire (pts (xy 34.925 240.03) (xy 33.02 240.03))
+  (wire (pts (xy 34.925 248.92) (xy 33.02 248.92))
     (stroke (width 0) (type solid) (color 0 0 0 0))
   )
@@
       (effects (font (size 1 1)))
     )
-    (property "Value" "Jumper_NO_Small" (id 1) (at 259.715 27.94 0)
+    (property "Value" "Jumper" (id 1) (at 259.715 27.94 0)
       (effects (font (size 1 1)) hide)
     )
@@
   (symbol (lib_id "Connector_Generic:Conn_01x03") (at 261.62 229.235 0) (unit 1)
     (in_bom yes) (on_board yes)
-    (property "Reference" "J10" (id 0) (at 260.35 223.5199 0)
+    (property "Reference" "J10" (id 0) (at 264.16 227.9649 0)
       (effects (font (size 1 1)) (justify left))
     )
-    (property "Value" "PJ392" (id 1) (at 264.795 232.4099 0)
-      (effects (font (size 1 1)) (justify left) hide)
+    (property "Value" "PJ-392" (id 1) (at 264.16 229.8699 0)
+      (effects (font (size 1 1)) (justify left))
     )
     (property "Footprint" "Connector_PinHeader_2.54mm:PinHeader_1x03_P2.54mm_Vertical" (id 2) (at 261.62 229.235 0)
@@
   (symbol (lib_id "Jumper:Jumper_3_Bridged12") (at 158.115 163.195 270) (unit 1)
     (in_bom yes) (on_board yes) (fields_autoplaced)
-    (property "Reference" "JP2" (id 0) (at 160.02 163.8299 90)
+    (property "Reference" "JP2" (id 0) (at 160.02 163.83 90)
       (effects (font (size 1 1)) (justify left))
     )
-    (property "Value" "Jumper_3_Bridged12" (id 1) (at 160.02 161.2901 90)
+    (property "Value" "Jumper" (id 1) (at 160.02 161.2901 90)
       (effects (font (size 1 1)) (justify left) hide)
     )
@@
       (effects (font (size 1 1)))
     )
-    (property "Value" "Conn_02x02_Odd_Even" (id 1) (at 306.705 137.16 0)
+    (property "Value" "Jumper" (id 1) (at 306.705 137.16 0)
       (effects (font (size 1 1)) hide)
     )
@@
       (effects (font (size 1 1)))
     )
-    (property "Footprint" "Crystal:Crystal_SMD_3225-4Pin_3.2x2.5mm_HandSoldering" (id 2) (at 260.35 183.515 0)
+    (property "Footprint" "Crystal:Crystal_SMD_SeikoEpson_TSX3225-4Pin_3.2x2.5mm_HandSoldering" (id 2) (at 260.35 183.515 0)
       (effects (font (size 1.27 1.27)) hide)
     )
@@
       (effects (font (size 1 1)) (justify left))
     )
-    (property "Value" "Pin header 1x6 Pitch=2.54mm" (id 1) (at 263.652 250.7996 0)
-      (effects (font (size 1 1)) (justify left) hide)
+    (property "Value" "MH-M18" (id 1) (at 263.652 250.7996 0)
+      (effects (font (size 1 1)) (justify left))
     )
     (property "Footprint" "Connector_PinHeader_2.54mm:PinHeader_1x06_P2.54mm_Vertical" (id 2) (at 261.62 248.285 0)
@@
       (effects (font (size 1.27 1.27)) hide)
     )
-    (property "Desc" "M18" (id 4) (at 263.652 250.7996 0)
-      (effects (font (size 1.27 1.27)) (justify left))
-    )
     (pin "1")
     (pin "2")
@@
   (symbol (lib_id "Connector:AudioJack4") (at 427.355 266.7 0) (mirror y) (unit 1)
     (in_bom yes) (on_board yes)
-    (property "Reference" "J14" (id 0) (at 427.355 261.62 0)
+    (property "Reference" "J14" (id 0) (at 427.355 259.715 0)
       (effects (font (size 1 1)) (justify right))
     )
-    (property "Value" "PJ-320" (id 1) (at 434.467 268.3764 0)
-      (effects (font (size 1 1)) (justify right) hide)
+    (property "Value" "PJ-320" (id 1) (at 426.212 261.3914 0)
+      (effects (font (size 1 1)) (justify right))
     )
     (property "Footprint" "my:PJ-320A_D" (id 2) (at 427.355 266.7 0)
@@
     )
     (path "/cae127c3-bfff-412b-9ec0-ee781bc1ac6e"
-      (reference "J9") (unit 1) (value "Conn_02x02_Odd_Even") (footprint "Connector_PinHeader_2.54mm:PinHeader_2x02_P2.54mm_Vertical")
+      (reference "J9") (unit 1) (value "Jumper") (footprint "Connector_PinHeader_2.54mm:PinHeader_2x02_P2.54mm_Vertical")
     )
     (path "/e8c4a248-1da0-4da0-82c3-044d513b286f"
-      (reference "J10") (unit 1) (value "PJ392") (footprint "Connector_PinHeader_2.54mm:PinHeader_1x03_P2.54mm_Vertical")
+      (reference "J10") (unit 1) (value "PJ-392") (footprint "Connector_PinHeader_2.54mm:PinHeader_1x03_P2.54mm_Vertical")
     )
     (path "/733e0df2-b5ba-4317-b4c0-8c3f642bd2b8"
@@
     )
     (path "/e9bf05b6-517e-43b4-9333-0db3a9fb1349"
-      (reference "J13") (unit 1) (value "Pin header 1x6 Pitch=2.54mm") (footprint "Connector_PinHeader_2.54mm:PinHeader_1x06_P2.54mm_Vertical")
+      (reference "J13") (unit 1) (value "MH-M18") (footprint "Connector_PinHeader_2.54mm:PinHeader_1x06_P2.54mm_Vertical")
     )
     (path "/7c2b712f-638f-4128-8ea8-d02c4be413f5"
@@
     )
     (path "/8d3b9c04-fa28-4334-9b75-a7b99c5601a1"
-      (reference "JP1") (unit 1) (value "Jumper_NO_Small") (footprint "Connector_PinHeader_2.54mm:PinHeader_1x02_P2.54mm_Vertical")
+      (reference "JP1") (unit 1) (value "Jumper") (footprint "Connector_PinHeader_2.54mm:PinHeader_1x02_P2.54mm_Vertical")
     )
     (path "/15565c30-e5ce-40db-bbdd-3aad7fd91675"
-      (reference "JP2") (unit 1) (value "Jumper_3_Bridged12") (footprint "Connector_PinHeader_2.54mm:PinHeader_1x03_P2.54mm_Vertical")
+      (reference "JP2") (unit 1) (value "Jumper") (footprint "Connector_PinHeader_2.54mm:PinHeader_1x03_P2.54mm_Vertical")
     )
     (path "/08b0dd2c-c8ff-4e18-bbd1-f3e29b12372f"
@@
     )
     (path "/1f0d16be-9630-4d59-b559-5e9a315adc32"
-      (reference "Y1") (unit 1) (value "12 MHz") (footprint "Crystal:Crystal_SMD_3225-4Pin_3.2x2.5mm_HandSoldering")
+      (reference "Y1") (unit 1) (value "12 MHz") (footprint "Crystal:Crystal_SMD_SeikoEpson_TSX3225-4Pin_3.2x2.5mm_HandSoldering")
     )
     (path "/5ee22c63-df9a-4ed7-b513-b77eefc1c114"

Commit message: update pcb rev.A
Parts:
- U7: symbol ad724:AD724 -> my:AD724
Changed lines of the file:
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@@
     (pin "9")
   )
-  (symbol (lib_id "ad724:AD724") (at 387.35 192.405 0) (unit 1)
+  (symbol (lib_id "my:AD724") (at 387.35 192.405 0) (unit 1)
     (in_bom yes) (on_board yes)
     (property "Reference" "U7" (id 0) (at 373.38 178.435 0)
