File: pcb_covers/rev.A/zxuno1010_covers.kicad_pcb (KiCad board)
At the start: 2 copper layers, 134.6 x 64 mm, 13 parts, among them J1 Mini-DIN-6, J11 TE 041021-4, J14 PJ-320, J16 USB_B_Micro, J2 Mini-DIN-6, J7 DB15_Female_HighDensity_Mount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, SW1 SW_Push, SW2 SW_Push, SW3 SW_Push

Commit message: update pcb covers rev.A
Parts:
- removed D1: LED_Red, LED_THT:LED_D3.0mm_Horizontal_O1.27mm_Z6.0mm
- removed D2: LED_Yellow, LED_THT:LED_D3.0mm_Horizontal_O1.27mm_Z6.0mm
- removed D3: LED_Green, LED_THT:LED_D3.0mm_Horizontal_O1.27mm_Z6.0mm
- removed J1, J2: Mini-DIN-6, my:MINI_DIN_6_33PRIMARY
- removed J11: TE 041021-4, my:SD_TE_2041021-mod
- removed J14: PJ-320, my:PJ-320A_D
- removed J16: USB_B_Micro, Connector_USB:USB_Micro-B_Molex-105017-0001
- removed J7: DB15_Female_HighDensity_MountingHoles, Connector_Dsub:DSUB-15-HD_Female_Horizontal_P2.29x1.98mm_EdgePinOffset3.03mm_Housed_MountingHolesOffset4.94mm
- removed SW1, SW2, SW3: SW_Push, Button_Switch_THT:SW_Tactile_SPST_Angled_PTS645Vx58-2LFS
